File: Electron/V2/PCB/EnvironmentMonitorV2.brd (EAGLE design)
At the start: 94 x 31.8 mm, 17 parts, among them U1 HTU21DSMD, U2 BMP180, U4 LIGHTSENSORTEMT6000

Commit message: Updated identifiers and added BOMs
Parts:
- R1: value 310R -> 1k5
- renumbered U$1 to U3
