File: Electron/V2/PCB/EnvironmentMonitorV2.sch (EAGLE design)
At the start: 17 parts, among them U1 HTU21DSMD, U2 BMP180, U4 LIGHTSENSORTEMT6000

Commit message: Updated identifiers and added BOMs
Parts:
- R1: value 310R -> 1k5
- renumbered U$1 to U3
Changed lines of the file:
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@@
 </classes>
 <parts>
-<part name="U$1" library="Tinamous" deviceset="ELECTRON" device="DUALNAMED"/>
+<part name="U3" library="Tinamous" deviceset="ELECTRON" device="DUALNAMED"/>
 <part name="JP1" library="Tinamous" deviceset="USB" device="A-SMD-MALE"/>
 <part name="SUPPLY1" library="SparkFun-Aesthetics" deviceset="5V" device=""/>
@@
 <part name="D1" library="SparkFun-DiscreteSemi" deviceset="DIODE" device="SMA"/>
 <part name="D2" library="SparkFun-LED" deviceset="LED" device="1206-BOTTOM"/>
-<part name="R1" library="SparkFun-Resistors" deviceset="RESISTOR" device="0805-RES" value="310R"/>
+<part name="R1" library="SparkFun-Resistors" deviceset="RESISTOR" device="0805-RES" value="1k5"/>
 <part name="GND8" library="SparkFun-Aesthetics" deviceset="GND" device=""/>
 </parts>
@@
 </plain>
 <instances>
-<instance part="U$1" gate="G$1" x="114.3" y="73.66"/>
+<instance part="U3" gate="G$1" x="114.3" y="73.66"/>
 <instance part="JP1" gate="G$1" x="35.56" y="68.58"/>
 <instance part="SUPPLY1" gate="G$1" x="20.32" y="91.44"/>
@@
 <net name="5V" class="0">
 <segment>
-<pinref part="U$1" gate="G$1" pin="VIN"/>
+<pinref part="U3" gate="G$1" pin="VIN"/>
 <pinref part="SUPPLY2" gate="G$1" pin="5V"/>
 <wire x1="104.14" y1="93.98" x2="93.98" y2="93.98" width="0.1524" layer="91"/>
@@
 <segment>
 <pinref part="GND2" gate="1" pin="GND"/>
-<pinref part="U$1" gate="G$1" pin="GND@2"/>
+<pinref part="U3" gate="G$1" pin="GND@2"/>
 <wire x1="86.36" y1="91.44" x2="104.14" y2="91.44" width="0.1524" layer="91"/>
 </segment>
 <segment>
 <pinref part="GND3" gate="1" pin="GND"/>
-<pinref part="U$1" gate="G$1" pin="GND"/>
+<pinref part="U3" gate="G$1" pin="GND"/>
 <wire x1="144.78" y1="86.36" x2="127" y2="86.36" width="0.1524" layer="91"/>
 </segment>
@@
 <net name="3.3V" class="0">
 <segment>
-<pinref part="U$1" gate="G$1" pin="3V3"/>
+<pinref part="U3" gate="G$1" pin="3V3"/>
 <pinref part="SUPPLY3" gate="G$1" pin="3.3V"/>
 <wire x1="127" y1="93.98" x2="137.16" y2="93.98" width="0.1524" layer="91"/>
@@
 <net name="N$1" class="0">
 <segment>
-<pinref part="U$1" gate="G$1" pin="!RST"/>
+<pinref part="U3" gate="G$1" pin="!RST"/>
 <wire x1="127" y1="91.44" x2="134.62" y2="91.44" width="0.1524" layer="91"/>
 </segment>
@@
 <net name="N$2" class="0">
 <segment>
-<pinref part="U$1" gate="G$1" pin="VBAT"/>
+<pinref part="U3" gate="G$1" pin="VBAT"/>
 <wire x1="127" y1="88.9" x2="134.62" y2="88.9" width="0.1524" layer="91"/>
 </segment>
@@
 <net name="OSHLED" class="0">
 <segment>
-<pinref part="U$1" gate="G$1" pin="D7"/>
+<pinref part="U3" gate="G$1" pin="D7"/>
 <wire x1="127" y1="83.82" x2="134.62" y2="83.82" width="0.1524" layer="91"/>
 <label x="134.62" y="83.82" size="1.27" layer="95" xref="yes"/>
@@
 <net name="N$4" class="0">
 <segment>
-<pinref part="U$1" gate="G$1" pin="D6"/>
+<pinref part="U3" gate="G$1" pin="D6"/>
 <wire x1="127" y1="81.28" x2="134.62" y2="81.28" width="0.1524" layer="91"/>
 </segment>
@@
 <net name="N$8" class="0">
 <segment>
-<pinref part="U$1" gate="G$1" pin="D2"/>
+<pinref part="U3" gate="G$1" pin="D2"/>
 <wire x1="127" y1="71.12" x2="134.62" y2="71.12" width="0.1524" layer="91"/>
 </segment>
@@
 <net name="SCL" class="0">
 <segment>
-<pinref part="U$1" gate="G$1" pin="D1"/>
+<pinref part="U3" gate="G$1" pin="D1"/>
 <wire x1="127" y1="68.58" x2="134.62" y2="68.58" width="0.1524" layer="91"/>
 <label x="134.62" y="68.58" size="1.016" layer="95" xref="yes"/>
@@
 <net name="SDA" class="0">
 <segment>
-<pinref part="U$1" gate="G$1" pin="D0"/>
+<pinref part="U3" gate="G$1" pin="D0"/>
 <wire x1="127" y1="66.04" x2="134.62" y2="66.04" width="0.1524" layer="91"/>
 <label x="134.62" y="66.04" size="1.016" layer="95" xref="yes"/>
@@
 <net name="N$11" class="0">
 <segment>
-<pinref part="U$1" gate="G$1" pin="C5"/>
+<pinref part="U3" gate="G$1" pin="C5"/>
 <wire x1="127" y1="63.5" x2="134.62" y2="63.5" width="0.1524" layer="91"/>
 </segment>
@@
 <net name="N$12" class="0">
 <segment>
-<pinref part="U$1" gate="G$1" pin="C4"/>
+<pinref part="U3" gate="G$1" pin="C4"/>
 <wire x1="127" y1="60.96" x2="134.62" y2="60.96" width="0.1524" layer="91"/>
 </segment>
@@
 <net name="N$13" class="0">
 <segment>
-<pinref part="U$1" gate="G$1" pin="C3"/>
+<pinref part="U3" gate="G$1" pin="C3"/>
 <wire x1="127" y1="58.42" x2="134.62" y2="58.42" width="0.1524" layer="91"/>
 </segment>
@@
 <net name="N$14" class="0">
 <segment>
-<pinref part="U$1" gate="G$1" pin="C2"/>
+<pinref part="U3" gate="G$1" pin="C2"/>
 <wire x1="127" y1="55.88" x2="134.62" y2="55.88" width="0.1524" layer="91"/>
 </segment>
@@
 <net name="N$15" class="0">
 <segment>
-<pinref part="U$1" gate="G$1" pin="C1"/>
+<pinref part="U3" gate="G$1" pin="C1"/>
 <wire x1="127" y1="53.34" x2="134.62" y2="53.34" width="0.1524" layer="91"/>
 </segment>
@@
 <net name="N$16" class="0">
 <segment>
-<pinref part="U$1" gate="G$1" pin="C0"/>
+<pinref part="U3" gate="G$1" pin="C0"/>
 <wire x1="127" y1="50.8" x2="134.62" y2="50.8" width="0.1524" layer="91"/>
 </segment>
@@
 <net name="N$17" class="0">
 <segment>
-<pinref part="U$1" gate="G$1" pin="B0"/>
+<pinref part="U3" gate="G$1" pin="B0"/>
 <wire x1="104.14" y1="50.8" x2="91.44" y2="50.8" width="0.1524" layer="91"/>
 </segment>
@@
 <net name="N$18" class="0">
 <segment>
-<pinref part="U$1" gate="G$1" pin="B1"/>
+<pinref part="U3" gate="G$1" pin="B1"/>
 <wire x1="104.14" y1="53.34" x2="91.44" y2="53.34" width="0.1524" layer="91"/>
 </segment>
@@
 <net name="N$19" class="0">
 <segment>
-<pinref part="U$1" gate="G$1" pin="B2"/>
+<pinref part="U3" gate="G$1" pin="B2"/>
 <wire x1="104.14" y1="55.88" x2="91.44" y2="55.88" width="0.1524" layer="91"/>
 </segment>
@@
 <net name="N$20" class="0">
 <segment>
-<pinref part="U$1" gate="G$1" pin="B3"/>
+<pinref part="U3" gate="G$1" pin="B3"/>
 <wire x1="104.14" y1="58.42" x2="91.44" y2="58.42" width="0.1524" layer="91"/>
 </segment>
@@
 <net name="N$21" class="0">
 <segment>
-<pinref part="U$1" gate="G$1" pin="B4"/>
+<pinref part="U3" gate="G$1" pin="B4"/>
 <wire x1="104.14" y1="60.96" x2="91.44" y2="60.96" width="0.1524" layer="91"/>
 </segment>
@@
 <net name="N$22" class="0">
 <segment>
-<pinref part="U$1" gate="G$1" pin="B5"/>
+<pinref part="U3" gate="G$1" pin="B5"/>
 <wire x1="104.14" y1="63.5" x2="91.44" y2="63.5" width="0.1524" layer="91"/>
 </segment>
@@
 <net name="N$25" class="0">
 <segment>
-<pinref part="U$1" gate="G$1" pin="A2"/>
+<pinref part="U3" gate="G$1" pin="A2"/>
 <wire x1="104.14" y1="71.12" x2="91.44" y2="71.12" width="0.1524" layer="91"/>
 </segment>
@@
 <net name="N$26" class="0">
 <segment>
-<pinref part="U$1" gate="G$1" pin="A3"/>
+<pinref part="U3" gate="G$1" pin="A3"/>
 <wire x1="104.14" y1="73.66" x2="91.44" y2="73.66" width="0.1524" layer="91"/>
 </segment>
@@
 <net name="N$27" class="0">
 <segment>
-<pinref part="U$1" gate="G$1" pin="A4"/>
+<pinref part="U3" gate="G$1" pin="A4"/>
 <wire x1="104.14" y1="76.2" x2="91.44" y2="76.2" width="0.1524" layer="91"/>
 </segment>
@@
 <net name="N$28" class="0">
 <segment>
-<pinref part="U$1" gate="G$1" pin="A5"/>
+<pinref part="U3" gate="G$1" pin="A5"/>
 <wire x1="104.14" y1="78.74" x2="91.44" y2="78.74" width="0.1524" layer="91"/>
 </segment>
@@
 <net name="N$29" class="0">
 <segment>
-<pinref part="U$1" gate="G$1" pin="DAC"/>
+<pinref part="U3" gate="G$1" pin="DAC"/>
 <wire x1="104.14" y1="81.28" x2="91.44" y2="81.28" width="0.1524" layer="91"/>
 </segment>
@@
 <net name="N$30" class="0">
 <segment>
-<pinref part="U$1" gate="G$1" pin="WKP"/>
+<pinref part="U3" gate="G$1" pin="WKP"/>
 <wire x1="104.14" y1="83.82" x2="91.44" y2="83.82" width="0.1524" layer="91"/>
 </segment>
@@
 <net name="N$31" class="0">
 <segment>
-<pinref part="U$1" gate="G$1" pin="RX"/>
+<pinref part="U3" gate="G$1" pin="RX"/>
 <wire x1="104.14" y1="86.36" x2="91.44" y2="86.36" width="0.1524" layer="91"/>
 </segment>
@@
 <net name="N$32" class="0">
 <segment>
-<pinref part="U$1" gate="G$1" pin="TX"/>
+<pinref part="U3" gate="G$1" pin="TX"/>
 <wire x1="104.14" y1="88.9" x2="91.44" y2="88.9" width="0.1524" layer="91"/>
 </segment>
@@
 <net name="INT" class="0">
 <segment>
-<pinref part="U$1" gate="G$1" pin="D3"/>
+<pinref part="U3" gate="G$1" pin="D3"/>
 <wire x1="127" y1="73.66" x2="134.62" y2="73.66" width="0.1524" layer="91"/>
 <label x="134.62" y="73.66" size="1.016" layer="95" xref="yes"/>
@@
 <net name="1WIRE-DQ" class="0">
 <segment>
-<pinref part="U$1" gate="G$1" pin="D5"/>
+<pinref part="U3" gate="G$1" pin="D5"/>
 <wire x1="127" y1="78.74" x2="134.62" y2="78.74" width="0.1524" layer="91"/>
 <label x="134.62" y="78.74" size="1.016" layer="95" xref="yes"/>
@@
 <net name="EXTERNAL_INT" class="0">
 <segment>
-<pinref part="U$1" gate="G$1" pin="D4"/>
+<pinref part="U3" gate="G$1" pin="D4"/>
 <wire x1="127" y1="76.2" x2="134.62" y2="76.2" width="0.1524" layer="91"/>
 <label x="134.62" y="76.2" size="1.016" layer="95" xref="yes"/>
@@
 <net name="UV_LEVEL" class="0">
 <segment>
-<pinref part="U$1" gate="G$1" pin="A0"/>
+<pinref part="U3" gate="G$1" pin="A0"/>
 <wire x1="104.14" y1="66.04" x2="91.44" y2="66.04" width="0.1524" layer="91"/>
 <label x="91.44" y="66.04" size="1.016" layer="95" rot="R180" xref="yes"/>
@@
 </segment>
 <segment>
-<pinref part="U$1" gate="G$1" pin="A1"/>
+<pinref part="U3" gate="G$1" pin="A1"/>
 <wire x1="104.14" y1="68.58" x2="91.44" y2="68.58" width="0.1524" layer="91"/>
 <label x="91.44" y="68.58" size="0.8128" layer="95" rot="R180" xref="yes"/>

Commit message: Updated software, added more values onto schematic.
Other:
- note added: "Stephen Harrison"
- note added: "V2.1"
- moved on the sheet: C4, R4
Changed lines of the file:
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@@
 <wire x1="160.02" y1="43.18" x2="243.84" y2="43.18" width="0.1524" layer="97"/>
 <wire x1="243.84" y1="43.18" x2="243.84" y2="106.68" width="0.1524" layer="97"/>
-<wire x1="243.84" y1="109.22" x2="243.84" y2="106.68" width="0.1524" layer="97"/>
 <wire x1="243.84" y1="106.68" x2="160.02" y2="106.68" width="0.1524" layer="97"/>
+<text x="238.76" y="7.62" size="1.778" layer="97">V2.1</text>
+<text x="165.862" y="11.684" size="1.778" layer="97">Stephen Harrison</text>
 </plain>
 <instances>
@@
 <instance part="GND4" gate="1" x="83.82" y="154.94"/>
 <instance part="R3" gate="G$1" x="172.72" y="157.48" rot="R180"/>
-<instance part="R4" gate="G$1" x="172.72" y="144.78" rot="R180"/>
+<instance part="R4" gate="G$1" x="172.72" y="149.86" rot="R180"/>
 <instance part="SUPPLY10" gate="G$1" x="162.56" y="160.02"/>
-<instance part="C4" gate="G$1" x="223.52" y="154.94" rot="R180"/>
+<instance part="C4" gate="G$1" x="63.5" y="167.64" rot="R180"/>
 <instance part="H1" gate="G$1" x="124.46" y="30.48"/>
 <instance part="H2" gate="G$1" x="124.46" y="22.86"/>
 <instance part="LOGO1" gate="G$1" x="223.52" y="93.98"/>
-<instance part="SUPPLY14" gate="G$1" x="223.52" y="160.02"/>
-<instance part="GND13" gate="1" x="223.52" y="144.78"/>
+<instance part="SUPPLY14" gate="G$1" x="63.5" y="172.72"/>
+<instance part="GND13" gate="1" x="63.5" y="157.48"/>
 <instance part="U4" gate="G$1" x="12.7" y="165.1"/>
 <instance part="R6" gate="G$1" x="15.24" y="147.32" rot="R90"/>
@@
 <instance part="SUPPLY6" gate="G$1" x="116.84" y="137.16"/>
 <instance part="C1" gate="G$1" x="134.62" y="132.08" rot="R180"/>
-<instance part="SUPPLY7" gate="G$1" x="134.62" y="142.24"/>
+<instance part="SUPPLY7" gate="G$1" x="134.62" y="137.16"/>
 <instance part="GND7" gate="1" x="134.62" y="121.92"/>
 <instance part="D1" gate="G$1" x="20.32" y="83.82" rot="R90"/>
@@
 <pinref part="C4" gate="G$1" pin="1"/>
 <pinref part="GND13" gate="1" pin="GND"/>
-<wire x1="223.52" y1="149.86" x2="223.52" y2="147.32" width="0.1524" layer="91"/>
+<wire x1="63.5" y1="162.56" x2="63.5" y2="160.02" width="0.1524" layer="91"/>
 </segment>
 <segment>
@@
 <wire x1="162.56" y1="157.48" x2="162.56" y2="160.02" width="0.1524" layer="91"/>
 <pinref part="R4" gate="G$1" pin="2"/>
-<wire x1="162.56" y1="157.48" x2="162.56" y2="144.78" width="0.1524" layer="91"/>
-<wire x1="162.56" y1="144.78" x2="167.64" y2="144.78" width="0.1524" layer="91"/>
+<wire x1="162.56" y1="157.48" x2="162.56" y2="149.86" width="0.1524" layer="91"/>
+<wire x1="162.56" y1="149.86" x2="167.64" y2="149.86" width="0.1524" layer="91"/>
 <junction x="162.56" y="157.48"/>
 </segment>
@@
 <pinref part="SUPPLY14" gate="G$1" pin="3.3V"/>
 <pinref part="C4" gate="G$1" pin="2"/>
-<wire x1="223.52" y1="160.02" x2="223.52" y2="157.48" width="0.1524" layer="91"/>
+<wire x1="63.5" y1="172.72" x2="63.5" y2="170.18" width="0.1524" layer="91"/>
 </segment>
 <segment>
@@
 <pinref part="C1" gate="G$1" pin="2"/>
 <pinref part="SUPPLY7" gate="G$1" pin="3.3V"/>
-<wire x1="134.62" y1="134.62" x2="134.62" y2="142.24" width="0.1524" layer="91"/>
+<wire x1="134.62" y1="134.62" x2="134.62" y2="137.16" width="0.1524" layer="91"/>
 </segment>
 </net>
@@
 <segment>
 <pinref part="R4" gate="G$1" pin="1"/>
-<wire x1="177.8" y1="144.78" x2="190.5" y2="144.78" width="0.1524" layer="91"/>
-<label x="190.5" y="144.78" size="1.016" layer="95" xref="yes"/>
+<wire x1="177.8" y1="149.86" x2="182.88" y2="149.86" width="0.1524" layer="91"/>
+<label x="182.88" y="149.86" size="1.016" layer="95" xref="yes"/>
 </segment>
 <segment>
@@
 <segment>
 <pinref part="R3" gate="G$1" pin="1"/>
-<wire x1="177.8" y1="157.48" x2="190.5" y2="157.48" width="0.1524" layer="91"/>
-<label x="190.5" y="157.48" size="1.016" layer="95" xref="yes"/>
+<wire x1="177.8" y1="157.48" x2="182.88" y2="157.48" width="0.1524" layer="91"/>
+<label x="182.88" y="157.48" size="1.016" layer="95" xref="yes"/>
 </segment>
 <segment>
@@
 <pinref part="U3" gate="G$1" pin="D3"/>
 <wire x1="127" y1="73.66" x2="134.62" y2="73.66" width="0.1524" layer="91"/>
-<label x="134.62" y="73.66" size="1.016" layer="95" xref="yes"/>
 </segment>
 </net>
@@
 <pinref part="U3" gate="G$1" pin="D5"/>
 <wire x1="127" y1="78.74" x2="134.62" y2="78.74" width="0.1524" layer="91"/>
-<label x="134.62" y="78.74" size="1.016" layer="95" xref="yes"/>
 </segment>
 </net>
@@
 <pinref part="U3" gate="G$1" pin="D4"/>
 <wire x1="127" y1="76.2" x2="134.62" y2="76.2" width="0.1524" layer="91"/>
-<label x="134.62" y="76.2" size="1.016" layer="95" xref="yes"/>
 </segment>
 </net>
@@
 <pinref part="U3" gate="G$1" pin="A0"/>
 <wire x1="104.14" y1="66.04" x2="91.44" y2="66.04" width="0.1524" layer="91"/>
-<label x="91.44" y="66.04" size="1.016" layer="95" rot="R180" xref="yes"/>
-</segment>
-</net>
+</segment>
+</net>
