File: Photon/V4.1/PCB/EnvironmentMonitorV4.1.brd (EAGLE design)
At the start: 55 x 32 mm, 29 parts, among them U5 CCS811, U6 BME280, U7 ALS-PT19, U8 ALS-PT19

Commit message: Updated library and set part values.
Parts:
- added D3: (no value), SparkFun-DiscreteSemi:SMA-DIODE
- added J1: (no value), SparkFun-Connectors:JST-2-SMD
- C2, C3: value 1.0uF -> 0.1uF
- R2, R5: value (none) -> 10k
- R3, R4: value (none) -> 4k7
- R6: value 100k -> 0R
- R8: value 4k7 -> 0R
- R9: value 100k -> 0
- moved C3 1.96 mm to (43.1, 4.81), turned to 90 degrees
- moved R2 1.73 mm to (46.3, 4.91), turned to 90 degrees
- moved R1 1.22 mm to (23.8, 2.18)
- moved D1 0.30 mm to (11.7, 2.64)
- moved LOGO1 0.06 mm to (50.0, 4.00)
Connections:
- new net N$4: D3.A, J1.2
- net GND: now also J1.1
- net V_USB: now also D3.C
- net WAKE: now also U$1.19
Routing:
- net WAKE: track 5.82 -> 30.3 mm, vias 0 -> 2
- net V_USB: track 3.47 -> 13.9 mm
- net LIGHTLEVEL_REAR: track 23.4 -> 15.6 mm
- net N$4: track 0.00 -> 4.85 mm, vias 0 -> 1
- net 3.3V: track 105.3 -> 102.6 mm
- net GND: track 2.32 -> 0.31 mm
- net LIGHTLEVEL_FRONT: track 30.4 -> 29.2 mm
- net N$6: track 28.6 -> 27.3 mm
- net OSHLED: track 2.79 -> 3.68 mm
Other:
- board text added: "+"
- board text added: "Max 5V DC"
