File: Feather/V6/PCB/EnvironmentMonitorV6.1.brd (EAGLE design)
At the start: 73 x 73 mm, 70 parts, among them IC1 BME680, IC2 TCS3472, IC3 CCS811, IC5 FEATHERWINGPADS_AND_PLACE_ONLY, Q1 IRFML8244TRPBF, Q2 4.3A/20V/54mΩ, U1 GRIDEYE, U2 LMV358, U3 LIS3DH

Commit message: Updates for V6.1
Parts:
- removed C16: 10uF, SparkFun-Capacitors:0805-CAP
- removed Q2: 4.3A/20V/54mΩ, SparkFun-DiscreteSemi:SOT23-3
- removed R13: 100R, SparkFun-Resistors:0805
- removed R23: 1M, SparkFun-Resistors:0805
- added J2: (no value), SparkFun-Connectors:1X05_1MM_RA
- added R24: DNP, SparkFun-Resistors:0805
- added R25: 0R, SparkFun-Resistors:0805
- added R27, R28: 10k, SparkFun-Resistors:0805
- R10, R21, R5, R9: value 10k -> DNP
- moved FRAME1 26.3 mm to (1.53, -11.8)
- moved C7 1.20 mm to (30.3, 52.6)
- moved C6 0.50 mm to (29.2, 56.6)
- moved J3 0.40 mm to (37.4, 44.3)
- moved C10 0.10 mm to (13.3, 63.0)
Connections:
- removed net N$10: Q2.1, R13.2, R23.2
- removed net N$21: C13.2, C14.2, Q2.3, U1.13, U1.9
- removed net N$3: IC3.4, IC3.5
- removed net OSHLED: IC5.12, R1.2
- new net AUX: IC3.8, R27.1, R28.2
- new net N$13: IC5.7, R25.2
- new net NTC_SENSE: IC3.4, IC3.5, R28.1
- new net SPI_MISO: IC5.13, J2.4
- new net SPI_MOSI: IC5.12, J2.3, R1.2
- new net SPI_SCK: IC5.11, J2.2
- net 3.3V: now also J2.5, R24.1, R27.2; no longer C16.2, Q2.2
- net GND: now also J2.1; no longer C16.1, R23.1
- net GRIDEYE_WAKE: now also C13.2, C14.2, U1.13, U1.9; no longer R13.1
- net VCCA: now also R24.2, R25.1; no longer IC5.7
Routing:
- net GRIDEYE_WAKE: track 71.1 -> 110.6 mm, vias 2 -> 4
- net 3.3V: track 335.2 -> 369.0 mm
- net N$21: track 25.9 -> 0.00 mm
- net SPI_MOSI: track 0.00 -> 20.4 mm
- net AUX: track 0.00 -> 18.9 mm, vias 0 -> 2
- net SPI_SCK: track 0.00 -> 17.9 mm
- net SPI_MISO: track 0.00 -> 10.9 mm
- net N$10: track 6.50 -> 0.00 mm
- net OSHLED: track 6.21 -> 0.00 mm
- net NTC_SENSE: track 0.00 -> 2.98 mm
- net VCCA: track 64.1 -> 61.3 mm
- net N$13: track 0.00 -> 2.51 mm
- net LIGHT_INT: track 122.5 -> 121.8 mm
- net N$3: track 0.60 -> 0.00 mm
- net CENTER_LED: track 17.3 -> 16.8 mm
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Other:
- board text added: "16 March 2019"
- board text added: "Low Power Option"
- board text added: "RCR123"
- board text added: "SPI"
- board text removed: "20 Feb 2019"
- board text removed: "CR123"
- board text removed: "Low Power Enable"
