File: Feather/V6/PCB/EnvironmentMonitorV6.1.sch (EAGLE design)
At the start: 70 parts, among them IC1 BME680, IC2 TCS3472, IC3 CCS811, IC5 FEATHERWINGPADS_AND_PLACE_ONLY, Q1 IRFML8244TRPBF, Q2 4.3A/20V/54mΩ, U1 GRIDEYE, U2 LMV358, U3 LIS3DH

Commit message: Updates for V6.1
Parts:
- removed C16: 10uF, SparkFun-Capacitors:1.0UF-25V-+80/-20(0805)"
- removed Q2: 4.3A/20V/54mΩ, SparkFun-DiscreteSemi:MOSFET_PCH-IRLML2244
- removed R13: 100R, SparkFun-Resistors:RESISTOR0805
- removed R23: 1M, SparkFun-Resistors:RESISTOR0805
- added J2: (no value), SparkFun-Connectors:CONN_05SMD2
- added R24: DNP, SparkFun-Resistors:RESISTOR0805
- added R25: 0R, SparkFun-Resistors:RESISTOR0805
- added R27, R28: 10k, SparkFun-Resistors:RESISTOR0805
- C18: FARNELL (none) -> 1457413; MFG (none) -> T491A106K010AT
- R10, R21, R5, R9: value 10k -> DNP
Connections:
- removed net N$10: Q2.G, R13.2, R23.2
- removed net N$21: C13.2, C14.2, Q2.D, U1.VDD, U1.VPP
- removed net N$3: IC3.PWM, IC3.SENSE
- removed net OSHLED: IC5.GPIOMOSI, R1.2
- new net AUX: IC3.AUX, R27.1, R28.2
- new net N$13: IC5.GPIOA2, R25.2
- new net NTC_SENSE: IC3.PWM, IC3.SENSE, R28.1
- new net SPI_MISO: IC5.GPIOMISO, J2.4
- new net SPI_MOSI: IC5.GPIOMOSI, J2.3, R1.2
- new net SPI_SCK: IC5.GPIOSCK, J2.2
- net 3.3V: now also J2.5, R24.1, R27.2; no longer C16.2, Q2.S
- net GND: now also J2.1; no longer C16.1, R23.1
- net GRIDEYE_WAKE: now also C13.2, C14.2, U1.VDD, U1.VPP; no longer R13.1
- net VCCA: now also R24.2, R25.1; no longer IC5.GPIOA2
Other:
- note added: "Accel @ 50Hz - removes 0.1-0.2mA"
- note added: "CCS_INT - During deep sleep is sourcing 1.5mA into Xenon"
- note added: "External Display SPI"
- note added: "Optional: 0R to power from 3v3 rail"
- note added: "Remove R10: Little difference"
- note added: "Remove R1: Little difference"
- note added: "Remove R25: Little difference"
- note added: "Remove R5: Little difference"
- note added: "V6.1 #1 and #2 PCBs using 100R"
- note added: "todo: resistor inline for int"
- note removed: "A0: PWM2 A1: PWM2 A2: PWM2 A3: PWM2 A4: PWM3"
- note removed: "Fit either C16 or C18"
- note removed: "This should be aluminium"
- moved on the sheet: C13, C14, C19, C5, C6, C7, D1, D3, J3, Q1, R15, R17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
