File: ArduinoNano33/V10/PCB/Environment-ArduinoNano44-Mini-Enclosure-V10-Top.sch (EAGLE design)
At the start: 19 parts, among them IC1 BME680

Commit message: Split out personal environmental sensor boards into individual Eagle files.
Parts:
- removed BT2, BT3: (no value), ThingySticks:BATTERY-12MM_PTH
- removed JP1: JUMPER-SMT_2_NC_PASTE_SILK, SparkFun-Jumpers:JUMPER-SMT_2_NC_PASTE_SILK
- removed JP2: USB-NEW-MICROB, Tinamous:USB-NEW-MICROB
- added D10, D11, D13, D14, D15, D16, D17, D18, D19, D22, D4, D5, D6, D7, D8, D9: Blue, ThingySticks:LED1206
- added D20, D21, D23: Green, ThingySticks:LED1206
- added J3, J6: (no value), SparkFun-Connectors:CONN_01
- added J4: QUIC, SparkFun-Connectors-2020-01-17:CONN_04SMD2
- added J5: (no value), SparkFun-Connectors-2020-01-17:USB_C2-LAYER
- added Q1, Q2: 5.8A/30V/35mΩ, SparkFun-DiscreteSemi:MOSFET-NCH-AO3404A
- added R10, R11, R12, R13, R14, R9: 1k5, SparkFun-Resistors:RESISTOR0805
- added R7: 5k1, SparkFun-Resistors:RESISTOR0805
- added S1: MOMENTARY-SWITCH-SPST-SMD-5.2MM, ThingySticks:MOMENTARY-SWITCH-SPST-SMD-5.2MM
- added U$6: (no value), ThingySticks:CR2032SMT
- added U$8, U$9: CR2032-SPLIT-PCBCR2032-NEGATIVE, ThingySticks:CR2032-SPLIT-PCBCR2032-NEGATIVE
- J1: device ThingySticks:CONN_02JST-2-PH-SIDE -> SparkFun-Connectors:CONN_01
- R2, R3: value 4k7 -> 1k5
- R6: value 1k5 -> 5k1
- U$1: value ARDUINO_33_NANOARDUINO_NANO_33_BLE_SENSE -> ARDUINO_33_NANOARDUINO_NANO_33_BLE_SENSE_SMD; device ThingySticks:ARDUINO_33_NANOARDUINO_NANO_33_BLE_SENSE -> ThingySticks:ARDUINO_33_NANOARDUINO_NANO_33_BLE_SENSE_SMD
Connections:
- removed net D5: R6.2, U$1.D5
- removed net D6: R5.2, U$1.D6
- removed net D9: R4.2, U$1.D9
- removed net V_BATT: BT2.+, BT3.+, JP1.2, U$1.VIN
- removed net V_USB: J1.1, JP2.VBUS, U$1.VUSB
- new net A: D18.A, D9.A, R13.1
- new net A0: S1.1, U$1.A0/DAC0
- new net B: D17.A, D21.A, D8.A, R12.1
- new net C: D11.A, D16.A, D7.A, R9.2
- new net CC1: J5.CC1, R7.1
- new net CC2: J5.CC2, R6.1
- new net D: D15.A, D23.A, D6.A, R10.2
- new net DIGIT1: D10.C, D4.C, D5.C, D6.C, D7.C, D8.C, D9.C, Q1.D
- new net DIGIT1_SELECT: Q1.G, U$1.A3
- new net DIGIT2: D13.C, D14.C, D15.C, D16.C, D17.C, D18.C, D19.C, Q2.D
- new net DIGIT2_SELECT: Q2.G, U$1.A6
- new net DIGIT3: D11.C, D20.C, D21.C, D22.C, D23.C, U$1.A7
- new net E: D14.A, D22.A, D5.A, R11.1
- new net F: D13.A, D4.A, R3.1
- new net G: D10.A, D19.A, D20.A, R2.1
- new net GREEN: R4.2, U$1.D6
- new net N$11: R10.1, U$1.A1
- new net N$12: R13.2, U$1.D2
- new net N$13: R3.2, U$1.D4
- new net N$4: D1.A, R14.1
- new net N$43: J3.1, U$1.D11/MOSI
- new net N$7: R9.1, U$1.A2
- new net N$8: R2.2, U$1.D13
- new net N$9: R11.2, U$1.D12/MISO
- new net NCF_ANTENNA1: J6.1, U$1.D8
- new net NCF_ANTENNA2: J1.1, U$1.D7
- new net RED: R14.2, U$1.D5
- new net SWITCH1: U$1.D10
- new net VIN: J5.VBUS, U$1.VIN
- new net YELLOW: R5.2, U$1.D9
- net 3.3V: now also J4.2, U$6.+1; no longer JP1.1, R2.2, R3.2
- net GND: now also J4.1, J5.GND, Q1.S, Q2.S, R6.2, R7.2, S1.2, U$6.-, U$8.-, U$9.-; no longer BT2.-, BT3.-, J1.2, JP2.GND
- net N$10: now also R12.2, U$1.D3; no longer D1.A, R6.1
- net SCL: now also J4.4; no longer R2.1
- net SDA: now also J4.3; no longer R3.1
Other:
- note added: "Avoid"
- note added: "Blue / White LEDs won't worn on a 3V CR battery."
- note added: "DP"
- note added: "Digit 3 Use: * B: Humidity * C: Q digit for Air Quality * D: Air Quality * E: DP * G: Temperature"
- note added: "For 3v Battery, go directly to 3v3 pin. Break 3v3 jumper on bottom of Arduino for low power operation."
- note added: "Humidity"
- note added: "If putting the batteries in series (i.e. to use blue LEDs / or for a high voltage), regulate to 3v3 or use VIn."
- note added: "NFC Antenna - Needs PCB Jumpers linked for D7/D8"
- note added: "Q"
- note added: "Temperature"
- note removed: "// Low power notes: // MP34DT05-A 1.6 - 3.6V. Tyical 1.8 (Mic) // LSM9DS3 1.9 V to 3.6 V (Accel) // APDS9960 2.4 - 3.6 (Typical 3.0) (Light) // LPS22HB 1.7 to 3.6 V (Pressure) // HTS221 1.7 to 3.6 V (Temperature / Humidity) // NINA-B3 1.7 to 3.6 (Typical 3.3) // DL3 - R + G + B LED (Blue won't work at 3v) // Extra... // BME680 1.71 to 3.6"
- note removed: "Arduino CPU: 4.2.3 Current consumption Table 14 shows the typical current consumption of a NINA-B3 module, independent of the software used. Mode Condition Typical Peak Sleep No clocks running, no RAM data retention 400 nA Sleep No clocks running, 64 kB RAM data retention 880 nA Sleep No clocks running, 256 kB RAM data retention 2.3 µA Standby RTC and 64 kB RAM data retention. System running on 3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"
- note removed: "CR2032: 3.0V, 210mAh Dropoff voltage, 2.5-2.0 Max current: 10mA CR2450: 15mA CR2016: 10mA CR1225: 3.0V, 48mAG Max 1.0mA"
- note removed: "Drive strngth. VCC >=2.7V Min 6, max 14ma. Typical 9mA"
- note removed: "Notes: Arduino has RGB LED. Do we need D1..D3. They could be right angle to project onto wall / floor / ceiling? Arduino needs 3v3 jumper broken on base - won't then use regulator to supply 3v3 so needs power (will battery work?) Add diode to batterys and direct to 3v3 supply, don't use VIN (V_BATT). V_IN will be disconnected Add option for external 3v3 supply (JST - bit not LiPol battery!) Remov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"
- moved on the sheet: D1, D2, D3, R2, R3, R4, R5, R6
